File: hw/ecp5_analog_video/ecp5_analog_video.kicad_pcb (KiCad board)
At the start: 4 copper layers, 80 x 46 mm, 62 parts, among them J1 ECP5EVB_VERSA, J2 DB15_Female_HighDensity_Mount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, J3 Barrel_Jack_Switch, J4 Mini-DIN-4, U1 ADV7123, U2 AD723

Commit message: Analog video board: update some resistor values.
Parts:
- R27, R28, R29: value 375R -> 374R
- R7: value 530R -> 536R
Changed lines of the file:
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@@
       (effects (font (size 0.61 0.61) (thickness 0.12)))
     )
-    (fp_text value 375R (at 0 0 90) (layer F.Fab)
+    (fp_text value 374R (at 0 0 90) (layer F.Fab)
       (effects (font (size 0.61 0.61) (thickness 0.12)))
     )
@@
       (effects (font (size 0.61 0.61) (thickness 0.12)))
     )
-    (fp_text value 375R (at 0 0 90) (layer F.Fab)
+    (fp_text value 374R (at 0 0 90) (layer F.Fab)
       (effects (font (size 0.61 0.61) (thickness 0.12)))
     )
@@
       (effects (font (size 0.61 0.61) (thickness 0.12)))
     )
-    (fp_text value 375R (at 0 0 90) (layer F.Fab)
+    (fp_text value 374R (at 0 0 90) (layer F.Fab)
       (effects (font (size 0.61 0.61) (thickness 0.12)))
     )
@@
       (effects (font (size 0.61 0.61) (thickness 0.12)))
     )
-    (fp_text value 530R (at 0 0 90) (layer F.Fab)
-      (effects (font (size 0.61 0.61) (thickness 0.12)))
-    )
+    (fp_text value 536R (at 0 0 90) (layer F.Fab)
+      (effects (font (size 0.61 0.61) (thickness 0.12)))
+    )
